Commit message: reduce max revolution of b1 thigh

File: resources/robots/b1/urdf/b1.urdf (robot description, URDF)
Before this commit: robot b1_description, 36 links, 35 joints
Joints:
- joint FL_thigh_joint: limit lower=-1.0 upper=3.5 effort=93.33 velocity=23.32 -> lower=-1.0 upper=2.0 effort=93.33 velocity=23.32
- joint FR_thigh_joint: limit lower=-1.0 upper=3.5 effort=93.33 velocity=23.32 -> lower=-1.0 upper=2.0 effort=93.33 velocity=23.32
- joint RL_thigh_joint: limit lower=-1.0 upper=3.5 effort=93.33 velocity=23.32 -> lower=-1.0 upper=2.0 effort=93.33 velocity=23.32
- joint RR_thigh_joint: limit lower=-1.0 upper=3.5 effort=93.33 velocity=23.32 -> lower=-1.0 upper=2.0 effort=93.33 velocity=23.32

Commit message: fixes to b1 urdf

File: resources/robots/b1/urdf/b1.urdf (robot description, URDF)
Before this commit: robot b1_description, 36 links, 35 joints
Links:
- link FL_hip: geometry visual mesh filename=../meshes/hipb.dae scale=1 1 1
- link FL_hip_rotor: geometry visual cylinder length=0.02 radius=0.05
- link FR_hip: geometry visual mesh filename=../meshes/hipb.dae scale=1 1 1
- link FR_hip_rotor: geometry visual cylinder length=0.02 radius=0.05
- link RL_hip: geometry visual mesh filename=../meshes/hipb.dae scale=1 1 1
- link RL_hip_rotor: geometry visual cylinder length=0.02 radius=0.05
- link RR_hip: geometry visual mesh filename=../meshes/hipb.dae scale=1 1 1
- link RR_hip_rotor: geometry visual cylinder length=0.02 radius=0.05
- link imu_link: geometry visual box size=0.001 0.001 0.001
